Commit message: fixes for kuka hw excitation

File: model/kuka_lwr4_stiffness.urdf (robot description, URDF)
Before this commit: robot single_lwr_robot, 9 links, 8 joints
Links:
- added link lwr_1_link_dummy
- added link lwr_2_link_dummy
- added link lwr_3_link_dummy
- added link lwr_4_link_dummy
- added link lwr_5_link_dummy
- added link lwr_6_link_dummy
- added link lwr_7_link_dummy
- link box: mass None -> 5.0
Joints:
- added joint lwr_0_joint_stiffness: type revolute, parent lwr_base_link, child lwr_1_link_dummy, axis 0 0 1, limit lower=0 upper=5000 effort=0 velocity=20000
- added joint lwr_1_joint_stiffness: type revolute, parent lwr_1_link, child lwr_2_link_dummy, axis 0 0 1, limit lower=0 upper=5000 effort=0 velocity=20000
- added joint lwr_2_joint_stiffness: type revolute, parent lwr_2_link, child lwr_3_link_dummy, axis 0 0 1, limit lower=0 upper=5000 effort=0 velocity=20000
- added joint lwr_3_joint_stiffness: type revolute, parent lwr_3_link, child lwr_4_link_dummy, axis 0 0 1, limit lower=0 upper=5000 effort=0 velocity=20000
- added joint lwr_4_joint_stiffness: type revolute, parent lwr_4_link, child lwr_5_link_dummy, axis 0 0 1, limit lower=0 upper=5000 effort=0 velocity=20000
- added joint lwr_5_joint_stiffness: type revolute, parent lwr_5_link, child lwr_6_link_dummy, axis 0 0 1, limit lower=0 upper=5000 effort=0 velocity=20000
- added joint lwr_6_joint_stiffness: type revolute, parent lwr_6_link, child lwr_7_link_dummy, axis 0 0 1, limit lower=0 upper=5000 effort=0 velocity=20000
