Commit message: random trajectory generation, fix WLS

File: model/kuka_lwr4_noisy_0.05.urdf (robot description, URDF)
Before this commit: robot single_lwr_robot, 9 links, 8 joints
Links:
- link lwr_1_link: mass 2.59505949714 -> 2.832425315
- link lwr_2_link: mass 2.64307710289 -> 2.6981578399
- link lwr_3_link: mass 2.77843455463 -> 2.64023810144
- link lwr_4_link: mass 2.67149058431 -> 2.7132577627
- link lwr_5_link: mass 1.68400461935 -> 1.73773034112
- link lwr_6_link: mass 1.6359384941 -> 1.56394365381
- link lwr_7_link: mass 0.281663251487 -> 0.382724970432
- link lwr_base_link: mass 1.59410424227 -> 1.58331084746
Joints:
- joint lwr_1_joint: origin xyz=0 0 0.2005 rpy=0 0 0 -> xyz=0.001 0.001 0.2005 rpy=0 0 0
