Commit message: simulate torques after reading in walking csv file, various other small fixes

File: model/bigman_robotran_right_leg.urdf (robot description, URDF)
Before this commit: robot bigman, 9 links, 8 joints
Links:
- link RFoot: mass 3.33109981 -> 3.83109981
- link RFootmot: mass 3.2844159 -> 2.2844159
- link RThighUpLeg: mass 3.2402068 -> 2.2402068
