Commit message: allow ignoring masses when identifying

File: model/kuka_lwr4.urdf (robot description, URDF)
Before this commit: robot single_lwr_robot, 9 links, 8 joints
Links:
- link lwr_1_link: mass 2.0 -> 2.7
- link lwr_2_link: mass 2.0 -> 2.7
- link lwr_3_link: mass 2.0 -> 2.7
- link lwr_4_link: mass 2.0 -> 2.7
- link lwr_5_link: mass 2.0 -> 1.7
- link lwr_6_link: mass 0.2 -> 1.6
- link lwr_7_link: mass 0.2 -> 0.3
- link lwr_base_link: mass 2.0 -> 2.7

Commit message: fix parameter output printing for some configurations, always use QR base regressor

File: model/kuka_lwr4.urdf (robot description, URDF)
Before this commit: robot single_lwr_robot, 9 links, 8 joints
Links:
- link lwr_base_link: mass 2.7 -> 1.6

Commit message: allow creating noisy urdf file

File: model/kuka_lwr4.urdf (robot description, URDF)
Before this commit: robot single_lwr_robot, 9 links, 8 joints
Links:
- link box: geometry collision box size=1.20 .74 1.0; visual box size=1.20 .74 1.0
Joints:
- joint box_lwr_base_joint: origin xyz=0 0 1 rpy=0 0 0 -> xyz=-0.25 0 1 rpy=0 0 0

Commit message: add full walkman meshes

File: model/kuka_lwr4.urdf (robot description, URDF)
Before this commit: robot single_lwr_robot, 9 links, 8 joints
Links:
- link lwr_1_link: geometry collision cylinder length=0.208 radius=0.07; collision sphere radius=0.07
- link lwr_2_link: geometry collision cylinder length=0.208 radius=0.07; collision sphere radius=0.07
- link lwr_3_link: geometry collision cylinder length=0.208 radius=0.07; collision sphere radius=0.07
- link lwr_4_link: geometry collision cylinder length=0.208 radius=0.07; collision sphere radius=0.07
- link lwr_5_link: geometry collision cylinder length=0.198 radius=0.07; collision sphere radius=0.07
- link lwr_6_link: geometry collision mesh filename=package://lwr_description/meshes/kuka/convex/arm_wrist_conv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; visual mesh filename=package://lwr_description/meshes/kuka/link_6.STL
- link lwr_7_link: geometry collision cylinder length=0.05 radius=0.04; visual mesh filename=package://lwr_description/meshes/kuka/link_7.STL
- link lwr_base_link: geometry collision cylinder length=0.11 radius=0.07; visual mesh filename=package://lwr_description/meshes/kuka/base.STL

File: model/walkman.urdf (robot description, URDF)
Before this commit: robot bigman, 85 links, 84 joints
Links:
- link DWL: geometry collision mesh filename=package://bigman_urdf/meshes/walkman/simple/TorsoRoll.STL scale=0.001 0.001 0.001; visual mesh filename=package://bigman_urdf/meshes/walkman/TorsoRoll.STL scale=0.001 0.001 0.001
- link DWS: geometry collision mesh filename=package://bigman_urdf/meshes/walkman/simple/TorsoYawPitch.S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 scale=0.001 0.001 0.001; visual mesh filename=package://bigman_urdf/meshes/walkman/TorsoYawPitch.STL scale=0.001 0.001 0.001
- link DWYTorso: geometry collision mesh filename=package://bigman_urdf/meshes/walkman/simple/NewChest.STL scale=0.001 0.001 0.001; visual mesh filename=package://bigman_urdf/meshes/walkman/NewChest.STL scale=0.001 0.001 0.001
- link LElb: geometry collision mesh filename=package://bigman_urdf/meshes/walkman/simple/Elbow.STL scale=0.001 -0.001 0.001; visual mesh filename=package://bigman_urdf/meshes/walkman/Elbow.STL scale=0.001 -0.001 0.001
- link LFoot: geometry collision box size=0.32 0.16 0.015; visual mesh filename=package://bigman_urdf/meshes/walkman/NewFoot.STL scale=0.001 -0.001 0.001
- link LFootmot: geometry collision mesh filename=package://bigman_urdf/meshes/walkman/simple/AnklePitch.STL scale=0.001 -0.001 0.001; visual mesh filename=package://bigman_urdf/meshes/walkman/AnklePitch.STL scale=0.001 -0.001 0.001
- link LForearm: geometry collision mesh filename=package://bigman_urdf/meshes/walkman/simple/Forearm.STL scale=0.001 -0.001 0.001; visual mesh filename=package://bigman_urdf/meshes/walkman/Forearm.STL scale=0.001 -0.001 0.001
- link LHipMot: geometry collision mesh filename=package://bigman_urdf/meshes/walkman/simple/HipRoll.STL scale=0.001 -0.001 0.001; visual mesh filename=package://bigman_urdf/meshes/walkman/HipRoll.STL scale=0.001 -0.001 0.001
- link LLowLeg: geometry collision mesh filename=package://bigman_urdf/meshes/walkman/simple/KneePitchCalf.S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 scale=0.001 -0.001 0.001; visual mesh filename=package://bigman_urdf/meshes/walkman/KneePitchCalf.STL scale=0.001 -0.001 0.001
- link LShp: geometry collision mesh filename=package://bigman_urdf/meshes/walkman/simple/ShoulderPitch.S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 scale=0.001 -0.001 0.001; visual mesh filename=package://bigman_urdf/meshes/walkman/ShoulderPitch.STL scale=0.001 -0.001 0.001
- link LShr: geometry collision mesh filename=package://bigman_urdf/meshes/walkman/simple/TopUpperArm.STL scale=0.001 -0.001 0.001; visual mesh filename=package://bigman_urdf/meshes/walkman/TopUpperArm.STL scale=0.001 -0.001 0.001
- link LShy: geometry collision mesh filename=package://bigman_urdf/meshes/walkman/simple/BottomUpperArm.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 scale=0.001 -0.001 0.001; visual mesh filename=package://bigman_urdf/meshes/walkman/BottomUpperArm.STL scale=0.001 -0.001 0.001
- link LSoftHandLink: geometry collision mesh filename=package://bigman_urdf/meshes/walkman/simple/SoftHandOpen.STL scale=0.001 -0.001 0.001; visual mesh filename=package://bigman_urdf/meshes/walkman/SoftHandOpen.STL scale=0.001 -0.001 0.001
- link LThighLowLeg: geometry collision mesh filename=package://bigman_urdf/meshes/walkman/simple/HipPitch.STL scale=0.001 -0.001 0.001; visual mesh filename=package://bigman_urdf/meshes/walkman/HipPitch.STL scale=0.001 -0.001 0.001
- link LThighUpLeg: geometry collision mesh filename=package://bigman_urdf/meshes/walkman/simple/HipYaw.STL scale=0.001 -0.001 0.001; visual mesh filename=package://bigman_urdf/meshes/walkman/HipYaw.STL scale=0.001 -0.001 0.001
- link LWrMot2: geometry collision mesh filename=package://bigman_urdf/meshes/walkman/simple/ForearmPitch.STL scale=0.001 -0.001 0.001; visual mesh filename=package://bigman_urdf/meshes/walkman/ForearmPitch.STL scale=0.001 -0.001 0.001
- link LWrMot3: geometry collision mesh filename=package://bigman_urdf/meshes/walkman/simple/ForearmRoll.STL scale=0.001 -0.001 0.001; visual mesh filename=package://bigman_urdf/meshes/walkman/ForearmRoll.STL scale=0.001 -0.001 0.001
- link NeckPitch: geometry collision mesh filename=package://bigman_urdf/meshes/walkman/simple/NeckPitch.STL scale=0.001 0.001 0.001; visual mesh filename=package://bigman_urdf/meshes/walkman/NeckPitch.STL scale=0.001 0.001 0.001
- link NeckYaw: geometry collision mesh filename=package://bigman_urdf/meshes/walkman/simple/NeckYaw.STL scale=0.001 0.001 0.001; visual mesh filename=package://bigman_urdf/meshes/walkman/NeckYaw.STL scale=0.001 0.001 0.001
- link RElb: geometry collision mesh filename=package://bigman_urdf/meshes/walkman/simple/Elbow.STL scale=0.001 0.001 0.001; visual mesh filename=package://bigman_urdf/meshes/walkman/Elbow.STL scale=0.001 0.001 0.001
- link RFoot: geometry collision box size=0.32 0.16 0.015; visual mesh filename=package://bigman_urdf/meshes/walkman/NewFoot.STL scale=0.001 0.001 0.001
- link RFootmot: geometry collision mesh filename=package://bigman_urdf/meshes/walkman/simple/AnklePitch.STL scale=0.001 0.001 0.001; visual mesh filename=package://bigman_urdf/meshes/walkman/AnklePitch.STL scale=0.001 0.001 0.001
- link RForearm: geometry collision mesh filename=package://bigman_urdf/meshes/walkman/simple/Forearm.STL scale=0.001 0.001 0.001; visual mesh filename=package://bigman_urdf/meshes/walkman/Forearm.STL scale=0.001 0.001 0.001
- link RHipMot: geometry collision mesh filename=package://bigman_urdf/meshes/walkman/simple/HipRoll.STL scale=0.001 0.001 0.001; visual mesh filename=package://bigman_urdf/meshes/walkman/HipRoll.STL scale=0.001 0.001 0.001
- link RLowLeg: geometry collision mesh filename=package://bigman_urdf/meshes/walkman/simple/KneePitchCalf.S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 scale=0.001 0.001 0.001; visual mesh filename=package://bigman_urdf/meshes/walkman/KneePitchCalf.STL scale=0.001 0.001 0.001
- link RShp: geometry collision mesh filename=package://bigman_urdf/meshes/walkman/simple/ShoulderPitch.S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 scale=0.001 0.001 0.001; visual mesh filename=package://bigman_urdf/meshes/walkman/ShoulderPitch.STL scale=0.001 0.001 0.001
- link RShr: geometry collision mesh filename=package://bigman_urdf/meshes/walkman/simple/TopUpperArm.STL scale=0.001 0.001 0.001; visual mesh filename=package://bigman_urdf/meshes/walkman/TopUpperArm.STL scale=0.001 0.001 0.001
- link RShy: geometry collision mesh filename=package://bigman_urdf/meshes/walkman/simple/BottomUpperArm.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 scale=0.001 0.001 0.001; visual mesh filename=package://bigman_urdf/meshes/walkman/BottomUpperArm.STL scale=0.001 0.001 0.001
- link RSoftHandLink: geometry collision mesh filename=package://bigman_urdf/meshes/walkman/simple/SoftHandOpen.STL scale=0.001 0.001 0.001; visual mesh filename=package://bigman_urdf/meshes/walkman/SoftHandOpen.STL scale=0.001 0.001 0.001
- link RThighLowLeg: geometry collision mesh filename=package://bigman_urdf/meshes/walkman/simple/HipPitch.STL scale=0.001 0.001 0.001; visual mesh filename=package://bigman_urdf/meshes/walkman/HipPitch.STL scale=0.001 0.001 0.001
- link RThighUpLeg: geometry collision mesh filename=package://bigman_urdf/meshes/walkman/simple/HipYaw.STL scale=0.001 0.001 0.001; visual mesh filename=package://bigman_urdf/meshes/walkman/HipYaw.STL scale=0.001 0.001 0.001
- link RWrMot2: geometry collision mesh filename=package://bigman_urdf/meshes/walkman/simple/ForearmPitch.STL scale=0.001 0.001 0.001; visual mesh filename=package://bigman_urdf/meshes/walkman/ForearmPitch.STL scale=0.001 0.001 0.001
- link RWrMot3: geometry collision mesh filename=package://bigman_urdf/meshes/walkman/simple/ForearmRoll.STL scale=0.001 0.001 0.001; visual mesh filename=package://bigman_urdf/meshes/walkman/ForearmRoll.STL scale=0.001 0.001 0.001
- link TorsoProtections: geometry collision mesh filename=package://bigman_urdf/meshes/walkman/simple/ProtectionSyste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 scale=0.001 0.001 0.001; visual mesh filename=package://bigman_urdf/meshes/walkman/ProtectionSystem.STL scale=0.001 0.001 0.001
- link Waist: geometry collision mesh filename=package://bigman_urdf/meshes/walkman/simple/Waist.STL scale=0.001 0.001 0.001; visual mesh filename=package://bigman_urdf/meshes/walkman/Waist.STL scale=0.001 0.001 0.001
- link multisense/head: geometry collision mesh filename=package://bigman_urdf/meshes/walkman/simple/Head.STL scale=0.001 0.001 0.001; visual mesh filename=package://bigman_urdf/meshes/walkman/Head.STL scale=0.001 0.001 0.001
- link multisense/hokuyo_link: geometry collision box size=0.08 0.06 0.04238; collision cylinder length=0.047 radius=0.024425
