Commit message: use rbdl as alternative to iDynTree for inverse dynamics

File: model/walkman_left_leg.urdf (robot description, URDF)
Before this commit: robot bigman, 9 links, 8 joints
Links:
- link LFoot: geometry collision box size=0.32 0.16 0.015; visual mesh filename=package://bigman_urdf/meshes/walkman/NewFoot.STL scale=0.001 -0.001 0.001
- link LFootmot: geometry collision mesh filename=package://bigman_urdf/meshes/walkman/simple/AnklePitch.STL scale=0.001 -0.001 0.001; visual mesh filename=package://bigman_urdf/meshes/walkman/AnklePitch.STL scale=0.001 -0.001 0.001
- link LHipMot: geometry collision mesh filename=package://bigman_urdf/meshes/walkman/simple/HipRoll.STL scale=0.001 -0.001 0.001; visual mesh filename=package://bigman_urdf/meshes/walkman/HipRoll.STL scale=0.001 -0.001 0.001
- link LLowLeg: geometry collision mesh filename=package://bigman_urdf/meshes/walkman/simple/KneePitchCalf.S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 scale=0.001 -0.001 0.001; visual mesh filename=package://bigman_urdf/meshes/walkman/KneePitchCalf.STL scale=0.001 -0.001 0.001
- link LThighLowLeg: geometry collision mesh filename=package://bigman_urdf/meshes/walkman/simple/HipPitch.STL scale=0.001 -0.001 0.001; visual mesh filename=package://bigman_urdf/meshes/walkman/HipPitch.STL scale=0.001 -0.001 0.001
- link LThighUpLeg: geometry collision mesh filename=package://bigman_urdf/meshes/walkman/simple/HipYaw.STL scale=0.001 -0.001 0.001; visual mesh filename=package://bigman_urdf/meshes/walkman/HipYaw.STL scale=0.001 -0.001 0.001
