Commit message: add rest of measured walkman links to table and urdf

File: model/walkman_orig.urdf (robot description, URDF)
Before this commit: robot bigman, 85 links, 84 joints
Links:
- link DWL: mass 1.635 -> 1.44965471
- link DWS: mass 6.7983647 -> 5.28825567
- link DWYTorso: mass 9.475 -> 26
- link LElb: mass 0.8898872 -> 8.6765385e-01
- link LFoot: mass 2.58 -> 3.42638110
- link LFootmot: mass 3.125 -> 3.2844159
- link LForearm: mass 2.17 -> 2.2127686
- link LHipMot: mass 4.2423495 -> 3.7958197
- link LLowLeg: mass 6.82012 -> 5.6495309
- link LShp: mass 1.93 -> 1.81745527
- link LShr: mass 5.5119737 -> 5.00486460
- link LShy: mass 3.1831391 -> 3.20289133
- link LSoftHandLink: mass 2.35 -> 1.2
- link LThighLowLeg: mass 5.31976 -> 5.0950736
- link LThighUpLeg: mass 3.06 -> 3.2402068
- link LWrMot2: mass 1.195 -> 1.2838072
- link LWrMot3: mass 0.175 -> 4.2801447e-01
- link NeckPitch: mass 0.18 -> 0.623
- link RElb: mass 0.8898872 -> 8.6765385e-01
- link RFoot: mass 2.58 -> 3.42638110
- link RFootmot: mass 3.125 -> 3.2844159
- link RForearm: mass 2.17 -> 2.2127686
- link RHipMot: mass 4.2423495 -> 3.7958197
- link RLowLeg: mass 6.82012 -> 5.6495309
- link RShp: mass 1.93 -> 1.81745527
- link RShr: mass 5.5119737 -> 5.00486460
- link RShy: mass 3.1831391 -> 3.20289133
- link RSoftHandLink: mass 2.35 -> 1.2
- link RThighLowLeg: mass 5.31976 -> 5.0950736
- link RThighUpLeg: mass 3.06 -> 3.2402068
- link RWrMot2: mass 1.195 -> 1.2838072
- link RWrMot3: mass 0.175 -> 4.2801447e-01
- link Waist: mass 11.2 -> 1.1046081e+01
- link backpack: mass None -> 10.0
- link multisense/hokuyo_link: mass 0.37 -> 0.057654
Joints:
- joint NeckPitchj: type fixed -> revolute
- joint NeckYawj: type fixed -> revolute
- joint WaistLat: type fixed -> revolute
