Commit message: some fixes and comments

File: model/kuka_lwr4_centroepiaggio.urdf (robot description, URDF)
Before this commit: robot single_lwr_robot, 16 links, 15 joints
Links:
- removed link lwr_1_link_dummy
- removed link lwr_2_link_dummy
- removed link lwr_3_link_dummy
- removed link lwr_4_link_dummy
- removed link lwr_5_link_dummy
- removed link lwr_6_link_dummy
- removed link lwr_7_link_dummy
- link box: mass 5.0 -> None; geometry collision box size=1.20 .74 1.0; visual box size=1.20 .74 1.0
- link lwr_1_link: mass 2.0 -> 2.7; geometry collision cylinder length=0.208 radius=0.07; collision sphere radius=0.07
- link lwr_2_link: mass 2.0 -> 2.7; geometry collision cylinder length=0.208 radius=0.07; collision sphere radius=0.07
- link lwr_3_link: mass 2.0 -> 2.7; geometry collision cylinder length=0.208 radius=0.07; collision sphere radius=0.07
- link lwr_4_link: mass 2.0 -> 2.7; geometry collision cylinder length=0.208 radius=0.07; collision sphere radius=0.07
- link lwr_5_link: mass 2.0 -> 1.7; geometry collision cylinder length=0.198 radius=0.07; collision sphere radius=0.07
- link lwr_6_link: mass 0.2 -> 1.1; geometry collision sphere radius=0.08; visual mesh filename=package://lwr_description/meshes/kuka/link_6.STL
- link lwr_7_link: mass 0.2 -> 0.25; geometry collision cylinder length=0.05 radius=0.04; visual mesh filename=package://lwr_description/meshes/kuka/link_7.STL
- link lwr_base_link: geometry collision cylinder length=0.11 radius=0.07; visual mesh filename=package://lwr_description/meshes/kuka/base.STL
Joints:
- removed joint lwr_0_joint_stiffness
- removed joint lwr_1_joint_stiffness
- removed joint lwr_2_joint_stiffness
- removed joint lwr_3_joint_stiffness
- removed joint lwr_4_joint_stiffness
- removed joint lwr_5_joint_stiffness
- removed joint lwr_6_joint_stiffness
- joint box_lwr_base_joint: origin xyz=0 0 1 rpy=0 0 0 -> xyz=-0.25 0 1 rpy=0 0 0
