Commit message: get constraint bounding boxes from STL files if specified in urdf (and files are present)

File: model/kuka_lwr4_cogimon.urdf (robot description, URDF)
Before this commit: robot kuka-lwr, 9 links, 8 joints
Links:
- link lwr_arm_1_link: geometry collision mesh filename=model://kuka-lwr-4plus/meshes/convex/arm_segment_a_convex.s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 scale=1.0 1.0 1.0; visual mesh filename=package://lwr_description/meshes/link_1.STL
- link lwr_arm_2_link: geometry collision mesh filename=model://kuka-lwr-4plus/meshes/convex/arm_segment_b_convex.s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 scale=1.0 1.0 1.0; visual mesh filename=package://lwr_description/meshes/link_2.STL
- link lwr_arm_3_link: geometry collision mesh filename=model://kuka-lwr-4plus/meshes/convex/arm_segment_a_convex.s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 scale=1.0 1.0 1.0; visual mesh filename=package://lwr_description/meshes/link_3.STL
- link lwr_arm_4_link: geometry collision mesh filename=model://kuka-lwr-4plus/meshes/convex/arm_segment_b_convex.s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 scale=1.0 1.0 1.0; visual mesh filename=package://lwr_description/meshes/link_4.STL
- link lwr_arm_5_link: geometry collision mesh filename=model://kuka-lwr-4plus/meshes/convex/arm_segment_last_conve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 scale=1.0 1.0 1.0; visual mesh filename=package://lwr_description/meshes/link_5.STL
- link lwr_arm_6_link: geometry collision mesh filename=model://kuka-lwr-4plus/meshes/convex/arm_wrist_convex.stl scale=1.0 1.0 1.0; visual mesh filename=package://lwr_description/meshes/link_6.STL
- link lwr_arm_7_link: geometry collision mesh filename=model://kuka-lwr-4plus/meshes/arm_flanche.dae scale=100 100 100; visual mesh filename=package://lwr_description/meshes/link_7.STL
- link lwr_arm_base_link: geometry collision mesh filename=model://kuka-lwr-4plus/meshes/convex/arm_base_convex.stl scale=0.9 0.9 0.9; visual mesh filename=package://lwr_description/meshes/base.STL

Commit message: fix displaying overall mass, some renames

File: model/kuka_lwr4_cogimon.urdf (robot description, URDF)
Before this commit: robot kuka-lwr, 9 links, 8 joints
Links:
- link lwr_arm_1_link: geometry collision mesh filename=model://kuka-lwr-4plus/meshes/convex/arm_segment_a_convex.s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 scale=1.0 1.0 1.0; visual mesh filename=package://lwr_description/meshes/kuka/link_1.STL
- link lwr_arm_2_link: geometry collision mesh filename=model://kuka-lwr-4plus/meshes/convex/arm_segment_b_convex.s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 scale=1.0 1.0 1.0; visual mesh filename=package://lwr_description/meshes/kuka/link_2.STL
- link lwr_arm_3_link: geometry collision mesh filename=model://kuka-lwr-4plus/meshes/convex/arm_segment_a_convex.s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 scale=1.0 1.0 1.0; visual mesh filename=package://lwr_description/meshes/kuka/link_3.STL
- link lwr_arm_4_link: geometry collision mesh filename=model://kuka-lwr-4plus/meshes/convex/arm_segment_b_convex.s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 scale=1.0 1.0 1.0; visual mesh filename=package://lwr_description/meshes/kuka/link_4.STL
- link lwr_arm_5_link: geometry collision mesh filename=model://kuka-lwr-4plus/meshes/convex/arm_segment_last_conve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 scale=1.0 1.0 1.0; visual mesh filename=package://lwr_description/meshes/kuka/link_5.STL
- link lwr_arm_6_link: geometry collision mesh filename=model://kuka-lwr-4plus/meshes/convex/arm_wrist_convex.stl scale=1.0 1.0 1.0; visual mesh filename=package://lwr_description/meshes/kuka/link_6.STL
- link lwr_arm_7_link: geometry collision mesh filename=model://kuka-lwr-4plus/meshes/arm_flanche.dae scale=100 100 100; visual mesh filename=package://lwr_description/meshes/kuka/link_7.STL
- link lwr_arm_base_link: geometry collision mesh filename=model://kuka-lwr-4plus/meshes/convex/arm_base_convex.stl scale=0.9 0.9 0.9; visual mesh filename=package://lwr_description/meshes/kuka/base.STL

Commit message: fixes

File: model/kuka_lwr4_cogimon.urdf (robot description, URDF)
Before this commit: robot kuka-lwr, 9 links, 8 joints
Links:
- removed link lwr_arm_1_link
- removed link lwr_arm_2_link
- removed link lwr_arm_3_link
- removed link lwr_arm_4_link
- removed link lwr_arm_5_link
- removed link lwr_arm_6_link
- removed link lwr_arm_7_link
- removed link lwr_arm_base_link
- added link lwr_1_link, mass 2.0; collision mesh filename=model://kuka-lwr-4plus/meshes/convex/arm_segment_a_convex.s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 scale=1.0 1.0 1.0; visual mesh filename=package://lwr_description/meshes/kuka/link_1.STL
- added link lwr_2_link, mass 2.0; collision mesh filename=model://kuka-lwr-4plus/meshes/convex/arm_segment_b_convex.s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 scale=1.0 1.0 1.0; visual mesh filename=package://lwr_description/meshes/kuka/link_2.STL
- added link lwr_3_link, mass 2.0; collision mesh filename=model://kuka-lwr-4plus/meshes/convex/arm_segment_a_convex.s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 scale=1.0 1.0 1.0; visual mesh filename=package://lwr_description/meshes/kuka/link_3.STL
- added link lwr_4_link, mass 2.0; collision mesh filename=model://kuka-lwr-4plus/meshes/convex/arm_segment_b_convex.s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 scale=1.0 1.0 1.0; visual mesh filename=package://lwr_description/meshes/kuka/link_4.STL
- added link lwr_5_link, mass 2.0; collision mesh filename=model://kuka-lwr-4plus/meshes/convex/arm_segment_last_conve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 scale=1.0 1.0 1.0; visual mesh filename=package://lwr_description/meshes/kuka/link_5.STL
- added link lwr_6_link, mass 1.0; collision mesh filename=model://kuka-lwr-4plus/meshes/convex/arm_wrist_convex.stl scale=1.0 1.0 1.0; visual mesh filename=package://lwr_description/meshes/kuka/link_6.STL
- added link lwr_7_link, mass 0.2; collision mesh filename=model://kuka-lwr-4plus/meshes/arm_flanche.dae scale=100 100 100; visual mesh filename=package://lwr_description/meshes/kuka/link_7.STL
- added link lwr_base_link, mass 1.2; collision mesh filename=model://kuka-lwr-4plus/meshes/convex/arm_base_convex.stl scale=0.9 0.9 0.9; visual mesh filename=package://lwr_description/meshes/kuka/base.STL
Joints:
- removed joint lwr_arm_0_joint
- removed joint lwr_arm_1_joint
- removed joint lwr_arm_2_joint
- removed joint lwr_arm_3_joint
- removed joint lwr_arm_4_joint
- removed joint lwr_arm_5_joint
- removed joint lwr_arm_6_joint
- added joint lwr_0_joint: type revolute, parent lwr_base_link, child lwr_1_link, origin xyz=0 0 0.11 rpy=0 0 0, axis 0 0 1, limit lower=-2.96705972839 upper=2.96705972839 effort=204 velocity=1.91986217719
- added joint lwr_1_joint: type revolute, parent lwr_1_link, child lwr_2_link, origin xyz=0 0 0.20 rpy=0 0 0, axis 0 -1 0, limit lower=-2.09439510239 upper=2.09439510239 effort=306 velocity=1.91986217719
- added joint lwr_2_joint: type revolute, parent lwr_2_link, child lwr_3_link, origin xyz=0 0 0.20 rpy=0 0 0, axis 0 0 1, limit lower=-2.96705972839 upper=2.96705972839 effort=204 velocity=2.26892802759
- added joint lwr_3_joint: type revolute, parent lwr_3_link, child lwr_4_link, origin xyz=0 0 0.20 rpy=0 0 0, axis 0 1 0, limit lower=-2.09439510239 upper=2.09439510239 effort=306 velocity=2.26892802759
- added joint lwr_4_joint: type revolute, parent lwr_4_link, child lwr_5_link, origin xyz=0 0 0.20 rpy=0 0 0, axis 0 0 1, limit lower=-2.96705972839 upper=2.96705972839 effort=204 velocity=2.26892802759
- added joint lwr_5_joint: type revolute, parent lwr_5_link, child lwr_6_link, origin xyz=0 0 0.19 rpy=0 0 0, axis 0 -1 0, limit lower=-2.09439510239 upper=2.09439510239 effort=306 velocity=3.14159265359
- added joint lwr_6_joint: type revolute, parent lwr_6_link, child lwr_7_link, origin xyz=0 0 0.078 rpy=0 0 0, axis 0 0 1, limit lower=-2.96705972839 upper=2.96705972839 effort=204 velocity=3.14159265359
- joint arm_world_joint: child lwr_arm_base_link -> lwr_base_link

Commit message: also give nrms error

File: model/kuka_lwr4_cogimon.urdf (robot description, URDF)
Before this commit: robot kuka-lwr, 9 links, 8 joints
Joints:
- joint lwr_0_joint: limit lower=-2.96705972839 upper=2.96705972839 effort=204 velocity=1.91986217719 -> lower=-2.96705972839 upper=2.96705972839 effort=176 velocity=1.91986217719
- joint lwr_1_joint: limit lower=-2.09439510239 upper=2.09439510239 effort=306 velocity=1.91986217719 -> lower=-2.09439510239 upper=2.09439510239 effort=176 velocity=1.91986217719
- joint lwr_2_joint: limit lower=-2.96705972839 upper=2.96705972839 effort=204 velocity=2.26892802759 -> lower=-2.96705972839 upper=2.96705972839 effort=100 velocity=2.26892802759
- joint lwr_3_joint: limit lower=-2.09439510239 upper=2.09439510239 effort=306 velocity=2.26892802759 -> lower=-2.09439510239 upper=2.09439510239 effort=100 velocity=2.26892802759
- joint lwr_4_joint: limit lower=-2.96705972839 upper=2.96705972839 effort=204 velocity=2.26892802759 -> lower=-2.96705972839 upper=2.96705972839 effort=100 velocity=2.26892802759
- joint lwr_5_joint: limit lower=-2.09439510239 upper=2.09439510239 effort=306 velocity=3.14159265359 -> lower=-2.09439510239 upper=2.09439510239 effort=38 velocity=3.14159265359
- joint lwr_6_joint: limit lower=-2.96705972839 upper=2.96705972839 effort=204 velocity=3.14159265359 -> lower=-2.96705972839 upper=2.96705972839 effort=38 velocity=3.14159265359
