Commit message: load meshes for visualizer, cache parsed xml files in helpers

File: model/twoLinks.urdf (robot description, URDF)
Before this commit: robot twoLinks, 3 links, 2 joints
Joints:
- joint joint_1_2: origin xyz=1 0 0 rpy=0 -0 0 -> xyz=0.5 0 0 rpy=0 0 0

File: model/walkman_only_legs.urdf (robot description, URDF)
Before this commit: robot bigman, 34 links, 33 joints
Links:
- link LFoot: geometry collision box size=0.32 0.16 0.015; visual mesh filename=package://bigman_urdf/meshes/walkman/NewFoot.STL scale=0.001 -0.001 0.001
- link LFootmot: geometry collision mesh filename=package://bigman_urdf/meshes/walkman/simple/AnklePitch.STL scale=0.001 -0.001 0.001; visual mesh filename=package://bigman_urdf/meshes/walkman/AnklePitch.STL scale=0.001 -0.001 0.001
- link LHipMot: geometry collision mesh filename=package://bigman_urdf/meshes/walkman/simple/HipRoll.STL scale=0.001 -0.001 0.001; visual mesh filename=package://bigman_urdf/meshes/walkman/HipRoll.STL scale=0.001 -0.001 0.001
- link LLowLeg: geometry collision mesh filename=package://bigman_urdf/meshes/walkman/simple/KneePitchCalf.S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 scale=0.001 -0.001 0.001; visual mesh filename=package://bigman_urdf/meshes/walkman/KneePitchCalf.STL scale=0.001 -0.001 0.001
- link LThighLowLeg: geometry collision mesh filename=package://bigman_urdf/meshes/walkman/simple/HipPitch.STL scale=0.001 -0.001 0.001; visual mesh filename=package://bigman_urdf/meshes/walkman/HipPitch.STL scale=0.001 -0.001 0.001
- link LThighUpLeg: geometry collision mesh filename=package://bigman_urdf/meshes/walkman/simple/HipYaw.STL scale=0.001 -0.001 0.001; visual mesh filename=package://bigman_urdf/meshes/walkman/HipYaw.STL scale=0.001 -0.001 0.001
- link PelvisWeightBench: geometry collision mesh filename=package://bigman_urdf/meshes/walkman/simple/PelvisWeightBen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 scale=0.001 0.001 0.001; visual mesh filename=package://bigman_urdf/meshes/walkman/PelvisWeightBench.STL scale=0.001 0.001 0.001
- link RFoot: geometry collision box size=0.32 0.16 0.015; visual mesh filename=package://bigman_urdf/meshes/walkman/NewFoot.STL scale=0.001 0.001 0.001
- link RFootmot: geometry collision mesh filename=package://bigman_urdf/meshes/walkman/simple/AnklePitch.STL scale=0.001 0.001 0.001; visual mesh filename=package://bigman_urdf/meshes/walkman/AnklePitch.STL scale=0.001 0.001 0.001
- link RHipMot: geometry collision mesh filename=package://bigman_urdf/meshes/walkman/simple/HipRoll.STL scale=0.001 0.001 0.001; visual mesh filename=package://bigman_urdf/meshes/walkman/HipRoll.STL scale=0.001 0.001 0.001
- link RLowLeg: geometry collision mesh filename=package://bigman_urdf/meshes/walkman/simple/KneePitchCalf.S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 scale=0.001 0.001 0.001; visual mesh filename=package://bigman_urdf/meshes/walkman/KneePitchCalf.STL scale=0.001 0.001 0.001
- link RThighLowLeg: geometry collision mesh filename=package://bigman_urdf/meshes/walkman/simple/HipPitch.STL scale=0.001 0.001 0.001; visual mesh filename=package://bigman_urdf/meshes/walkman/HipPitch.STL scale=0.001 0.001 0.001
- link RThighUpLeg: geometry collision mesh filename=package://bigman_urdf/meshes/walkman/simple/HipYaw.STL scale=0.001 0.001 0.001; visual mesh filename=package://bigman_urdf/meshes/walkman/HipYaw.STL scale=0.001 0.001 0.001
- link Waist: geometry collision mesh filename=package://bigman_urdf/meshes/walkman/simple/Waist.STL scale=0.001 0.001 0.001; visual mesh filename=package://bigman_urdf/meshes/walkman/Waist.STL scale=0.001 0.001 0.001
