Commit message: fixes

File: model/threeLinks.urdf (robot description, URDF)
Before this commit: robot twoLinks, 4 links, 3 joints
Links:
- added link contact_ft
Joints:
- added joint contact_ft_joint: type fixed, parent link2, child contact_ft, origin xyz=0 0 0.1 rpy=0 0 0

Commit message: use default 'python' excutable (not python3)

File: model/threeLinks.urdf (robot description, URDF)
Before this commit: robot twoLinks, 5 links, 4 joints
Links:
- link link1: geometry collision box size=0.5 0.5 0.5; visual box size=0.5 0.5 0.5
- link link2: geometry collision box size=0.5 0.5 0.5; visual box size=0.5 0.5 0.5
- link link3: geometry collision box size=0.5 0.5 0.5; visual box size=0.5 0.5 0.5

Commit message: use bounding box offset if using geometry from urdf

File: model/threeLinks.urdf (robot description, URDF)
Before this commit: robot twoLinks, 5 links, 4 joints
Links:
- link link1: geometry collision box size=0.5 0.1 0.1; visual box size=0.5 0.1 0.1
- link link2: geometry collision box size=0.5 0.1 0.1; visual box size=0.5 0.1 0.1
- link link3: geometry collision box size=0.5 0.1 0.1; visual box size=0.5 0.1 0.1
Joints:
- joint joint_1_2: origin xyz=1 0 0 rpy=0 -0 0 -> xyz=0.25 0 0 rpy=0 -0 0
- joint joint_2_3: axis 0 0 1 -> 0 1 0.5; origin xyz=1 0 0 rpy=0 -0 0 -> xyz=0.25 0 0 rpy=0 -0 0

Commit message: add simulator for generated trajectories

File: model/threeLinks.urdf (robot description, URDF)
Before this commit: robot twoLinks, 5 links, 4 joints
Joints:
- joint joint_1_2: origin xyz=0.25 0 0 rpy=0 -0 0 -> xyz=0.5 0 0 rpy=0 -0 0
- joint joint_2_3: origin xyz=0.25 0 0 rpy=0 -0 0 -> xyz=0.5 0 0 rpy=0 -0 0
