Commit message: add bounded trajectory generation to prevent running into angle limits
* various fixes
* allows trajectory generation for single walkman arm
* also visualizer improvements: show collisions, convex hull, torques

File: model/walkman_left_arm.urdf (robot description, URDF)
Before this commit: robot bigman, 13 links, 12 joints
Links:
- link LElb: geometry collision mesh filename=package://bigman_urdf/meshes/walkman/simple/Elbow.STL scale=0.001 -0.001 0.001; visual mesh filename=package://bigman_urdf/meshes/walkman/Elbow.STL scale=0.001 -0.001 0.001
- link LForearm: geometry collision mesh filename=package://bigman_urdf/meshes/walkman/simple/Forearm.STL scale=0.001 -0.001 0.001; visual mesh filename=package://bigman_urdf/meshes/walkman/Forearm.STL scale=0.001 -0.001 0.001
- link LShp: geometry collision mesh filename=package://bigman_urdf/meshes/walkman/simple/ShoulderPitch.S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 scale=0.001 -0.001 0.001; visual mesh filename=package://bigman_urdf/meshes/walkman/ShoulderPitch.STL scale=0.001 -0.001 0.001
- link LShr: geometry collision mesh filename=package://bigman_urdf/meshes/walkman/simple/TopUpperArm.STL scale=0.001 -0.001 0.001; visual mesh filename=package://bigman_urdf/meshes/walkman/TopUpperArm.STL scale=0.001 -0.001 0.001
- link LShy: geometry collision mesh filename=package://bigman_urdf/meshes/walkman/simple/BottomUpperArm.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 scale=0.001 -0.001 0.001; visual mesh filename=package://bigman_urdf/meshes/walkman/BottomUpperArm.STL scale=0.001 -0.001 0.001
- link LSoftHandLink: geometry collision mesh filename=package://bigman_urdf/meshes/walkman/simple/SoftHandOpen.STL scale=0.001 -0.001 0.001; visual mesh filename=package://bigman_urdf/meshes/walkman/SoftHandOpen.STL scale=0.001 -0.001 0.001
- link LWrMot2: geometry collision mesh filename=package://bigman_urdf/meshes/walkman/simple/ForearmPitch.STL scale=0.001 -0.001 0.001; visual mesh filename=package://bigman_urdf/meshes/walkman/ForearmPitch.STL scale=0.001 -0.001 0.001
- link LWrMot3: geometry collision mesh filename=package://bigman_urdf/meshes/walkman/simple/ForearmRoll.STL scale=0.001 -0.001 0.001; visual mesh filename=package://bigman_urdf/meshes/walkman/ForearmRoll.STL scale=0.001 -0.001 0.001
- link Waist: geometry collision mesh filename=package://bigman_urdf/meshes/walkman/simple/Waist.STL scale=0.001 0.001 0.001; visual mesh filename=package://bigman_urdf/meshes/walkman/Waist.STL scale=0.001 0.001 0.001

File: model/world_walkman_fixed.urdf (robot description, URDF)
Before this commit: robot ground, 3 links, 1 joints
Links:
- link ground_link: geometry visual box size=5.0 5.0 0.05
- link seat_link: geometry visual box size=.08 .035 1.275
