Commit message: fix urdf with measured weights

File: model/walkman_measured.urdf (robot description, URDF)
Before this commit: robot bigman, 85 links, 84 joints
Links:
- link NeckYaw: mass 0.35 -> 0.555
- link backpack: mass None -> 15.0
- link multisense/head: mass 1.41984 -> 4.105

Commit message: fixes for gravity only identification, allow using data regressor directly to determine base dependencies, allow rbdl with floating-base

File: model/walkman_measured.urdf (robot description, URDF)
Before this commit: robot bigman, 85 links, 84 joints
Links:
- added link crane_ft
Joints:
- added joint crane_ft_joint: type fixed, parent DWYTorso, child crane_ft, origin xyz=0 0 0.480 rpy=0 0 0

Commit message: performance improvements

File: model/walkman_measured.urdf (robot description, URDF)
Before this commit: robot bigman, 86 links, 85 joints
Joints:
- joint LAnkLat: limit lower=-0.785 upper=0.785 effort=120 velocity=6.283 -> lower=-0.785 upper=0.785 effort=210 velocity=16.7
- joint LAnkSag: limit lower=-1.39556 upper=0.697778 effort=220 velocity=6.283 -> lower=-1.39556 upper=0.697778 effort=330 velocity=18.6
- joint LElbj: limit lower=-2.96705972838 upper=0.593411945677 effort=120 velocity=6.283 -> lower=-2.96705972838 upper=0.593411945677 effort=56 velocity=11.3
- joint LForearmPlate: limit lower=-2.529 upper=2.529 effort=60 velocity=6.283 -> lower=-2.529 upper=2.529 effort=56 velocity=11.3
- joint LHipLat: limit lower=-0.697778 upper=0.87222 effort=220 velocity=6.283 -> lower=-0.697778 upper=0.87222 effort=400 velocity=9.0
- joint LHipSag: limit lower=-2.09333 upper=1.046667 effort=220 velocity=6.283 -> lower=-2.09333 upper=1.046667 effort=400 velocity=8.2
- joint LHipYaw: limit lower=-0.872222 upper=1.57 effort=120 velocity=6.283 -> lower=-0.872222 upper=1.57 effort=140 velocity=19.5
- joint LKneeSag: limit lower=0.0 upper=2.442222 effort=220 velocity=6.283 -> lower=0.0 upper=2.442222 effort=400 velocity=8.2
- joint LShLat: limit lower=0.0872664625995 upper=3.8571776469 effort=120 velocity=6.283 -> lower=0.0872664625995 upper=3.8571776469 effort=140 velocity=16.7
- joint LShSag: limit lower=-2.87979326578 upper=2.79252680318 effort=60 velocity=6.283 -> lower=-2.87979326578 upper=2.79252680318 effort=140 velocity=16.7
- joint LShYaw: limit lower=-2.84488668074 upper=2.84488668074 effort=120 velocity=6.283 -> lower=-2.84488668074 upper=2.84488668074 effort=140 velocity=16.7
- joint LWrj1: limit lower=-1.48 upper=1.48 effort=60 velocity=6.283 -> lower=-1.48 upper=1.48 effort=56 velocity=11.3
- joint LWrj2: limit lower=-1.48 upper=1.48 effort=60 velocity=6.283 -> lower=-1.48 upper=1.48 effort=56 velocity=11.3
- joint RAnkLat: limit lower=-0.785 upper=0.785 effort=120 velocity=6.283 -> lower=-0.785 upper=0.785 effort=210 velocity=16.7
- joint RAnkSag: limit lower=-1.39556 upper=0.697778 effort=220 velocity=6.283 -> lower=-1.39556 upper=0.697778 effort=330 velocity=18.6
- joint RElbj: limit lower=-2.96705972838 upper=0.593411945677 effort=60 velocity=6.283 -> lower=-2.96705972838 upper=0.593411945677 effort=56 velocity=11.3
- joint RForearmPlate: limit lower=-2.529 upper=2.529 effort=60 velocity=6.283 -> lower=-2.529 upper=2.529 effort=56 velocity=11.3
- joint RHipLat: limit lower=-0.87222 upper=0.697778 effort=220 velocity=6.283 -> lower=-0.87222 upper=0.697778 effort=400 velocity=9.0
- joint RHipSag: limit lower=-2.09333 upper=1.046667 effort=220 velocity=6.283 -> lower=-2.09333 upper=1.046667 effort=400 velocity=8.2
- joint RHipYaw: limit lower=-1.57 upper=0.872222 effort=120 velocity=6.283 -> lower=-1.57 upper=0.872222 effort=140 velocity=19.5
- joint RKneeSag: limit lower=0.0 upper=2.442222 effort=220 velocity=6.283 -> lower=0.0 upper=2.442222 effort=400 velocity=8.2
- joint RShLat: limit lower=-3.8571776469 upper=-0.122173047639 effort=120 velocity=6.283 -> lower=-3.8571776469 upper=-0.122173047639 effort=140 velocity=16.7
- joint RShSag: limit lower=-2.84488668074 upper=2.8099800957 effort=120 velocity=6.283 -> lower=-2.84488668074 upper=2.8099800957 effort=140 velocity=16.7
- joint RShYaw: limit lower=-2.86233997326 upper=2.82743338822 effort=120 velocity=6.283 -> lower=-2.86233997326 upper=2.82743338822 effort=140 velocity=16.7
- joint RWrj1: limit lower=-1.48 upper=1.48 effort=60 velocity=6.283 -> lower=-1.48 upper=1.48 effort=56 velocity=11.3
- joint RWrj2: limit lower=-1.48 upper=1.48 effort=60 velocity=6.283 -> lower=-1.48 upper=1.48 effort=56 velocity=11.3
- joint WaistLat: limit lower=-0.3490658503988659 upper=0.3490658503988659 effort=120 velocity=6.283 -> lower=-0.3490658503988659 upper=0.3490658503988659 effort=210 velocity=16.7
- joint WaistSag: limit lower=-0.349065850398 upper=1.39626340159 effort=220 velocity=6.283 -> lower=-0.349065850398 upper=1.39626340159 effort=400 velocity=9.0
- joint WaistYaw: limit lower=-2.84488668074 upper=2.84488668074 effort=120 velocity=6.283 -> lower=-2.84488668074 upper=2.84488668074 effort=140 velocity=19.5
