Commit message: ignore some fixated walkman links (for current dataset)

File: model/walkman.urdf (robot description, URDF)
Before this commit: robot bigman, 85 links, 84 joints
Joints:
- joint NeckPitchj: type revolute -> fixed
- joint NeckYawj: type revolute -> fixed
- joint WaistLat: type revolute -> fixed

Commit message: allow generating static trajectories for identification of gravity terms, fixes for floating base, some small updates for walkman urdfs (from main repo)

File: model/walkman.urdf (robot description, URDF)
Before this commit: robot bigman, 85 links, 84 joints
Links:
- added link crane_ft
Joints:
- added joint crane_ft_joint: type fixed, parent DWYTorso, child crane_ft, origin xyz=0 0 0.480 rpy=0 0 0
- joint LAnkLat: limit lower=-0.785 upper=0.785 effort=210 velocity=6.283 -> lower=-0.785 upper=0.785 effort=120 velocity=6.283
- joint LAnkSag: limit lower=-1.39556 upper=0.697778 effort=330 velocity=6.283 -> lower=-1.39556 upper=0.697778 effort=220 velocity=6.283
- joint LHipLat: limit lower=-0.697778 upper=0.87222 effort=400 velocity=6.283 -> lower=-0.697778 upper=0.87222 effort=220 velocity=6.283
- joint LHipSag: limit lower=-2.09333 upper=1.046667 effort=400 velocity=6.283 -> lower=-2.09333 upper=1.046667 effort=220 velocity=6.283
- joint LHipYaw: limit lower=-0.872222 upper=1.57 effort=140 velocity=6.283 -> lower=-0.872222 upper=1.57 effort=120 velocity=6.283
- joint LKneeSag: limit lower=0.0 upper=2.442222 effort=400 velocity=6.283 -> lower=0.0 upper=2.442222 effort=220 velocity=6.283
- joint LShSag: limit lower=-2.87979326578 upper=2.79252680318 effort=120 velocity=6.283 -> lower=-2.87979326578 upper=2.79252680318 effort=60 velocity=6.283
- joint NeckPitchj: origin xyz=0 0 0.117 rpy=0 0 0 -> xyz=0 0 0.1155 rpy=0 0 0
- joint RAnkLat: limit lower=-0.785 upper=0.785 effort=210 velocity=6.283 -> lower=-0.785 upper=0.785 effort=120 velocity=6.283
- joint RAnkSag: limit lower=-1.39556 upper=0.697778 effort=330 velocity=6.283 -> lower=-1.39556 upper=0.697778 effort=220 velocity=6.283
- joint RElbj: limit lower=-2.96705972838 upper=0.593411945677 effort=120 velocity=6.283 -> lower=-2.96705972838 upper=0.593411945677 effort=60 velocity=6.283
- joint RHipLat: limit lower=-0.87222 upper=0.697778 effort=400 velocity=6.283 -> lower=-0.87222 upper=0.697778 effort=220 velocity=6.283
- joint RHipSag: limit lower=-2.09333 upper=1.046667 effort=400 velocity=6.283 -> lower=-2.09333 upper=1.046667 effort=220 velocity=6.283
- joint RHipYaw: limit lower=-1.57 upper=0.872222 effort=140 velocity=6.283 -> lower=-1.57 upper=0.872222 effort=120 velocity=6.283
- joint RKneeSag: limit lower=0.0 upper=2.442222 effort=400 velocity=6.283 -> lower=0.0 upper=2.442222 effort=220 velocity=6.283

File: model/walkman_measured.urdf (robot description, URDF)
Before this commit: robot bigman, 85 links, 84 joints
Joints:
- joint LAnkLat: limit lower=-0.785 upper=0.785 effort=210 velocity=6.283 -> lower=-0.785 upper=0.785 effort=120 velocity=6.283
- joint LAnkSag: limit lower=-1.39556 upper=0.697778 effort=330 velocity=6.283 -> lower=-1.39556 upper=0.697778 effort=220 velocity=6.283
- joint LHipLat: limit lower=-0.697778 upper=0.87222 effort=400 velocity=6.283 -> lower=-0.697778 upper=0.87222 effort=220 velocity=6.283
- joint LHipSag: limit lower=-2.09333 upper=1.046667 effort=400 velocity=6.283 -> lower=-2.09333 upper=1.046667 effort=220 velocity=6.283
- joint LHipYaw: limit lower=-0.872222 upper=1.57 effort=140 velocity=6.283 -> lower=-0.872222 upper=1.57 effort=120 velocity=6.283
- joint LKneeSag: limit lower=0.0 upper=2.442222 effort=400 velocity=6.283 -> lower=0.0 upper=2.442222 effort=220 velocity=6.283
- joint LShSag: limit lower=-2.87979326578 upper=2.79252680318 effort=120 velocity=6.283 -> lower=-2.87979326578 upper=2.79252680318 effort=60 velocity=6.283
- joint NeckPitchj: origin xyz=0 0 0.117 rpy=0 0 0 -> xyz=0 0 0.1155 rpy=0 0 0
- joint RAnkLat: limit lower=-0.785 upper=0.785 effort=210 velocity=6.283 -> lower=-0.785 upper=0.785 effort=120 velocity=6.283
- joint RAnkSag: limit lower=-1.39556 upper=0.697778 effort=330 velocity=6.283 -> lower=-1.39556 upper=0.697778 effort=220 velocity=6.283
- joint RElbj: limit lower=-2.96705972838 upper=0.593411945677 effort=120 velocity=6.283 -> lower=-2.96705972838 upper=0.593411945677 effort=60 velocity=6.283
- joint RHipLat: limit lower=-0.87222 upper=0.697778 effort=400 velocity=6.283 -> lower=-0.87222 upper=0.697778 effort=220 velocity=6.283
- joint RHipSag: limit lower=-2.09333 upper=1.046667 effort=400 velocity=6.283 -> lower=-2.09333 upper=1.046667 effort=220 velocity=6.283
- joint RHipYaw: limit lower=-1.57 upper=0.872222 effort=140 velocity=6.283 -> lower=-1.57 upper=0.872222 effort=120 velocity=6.283
- joint RKneeSag: limit lower=0.0 upper=2.442222 effort=400 velocity=6.283 -> lower=0.0 upper=2.442222 effort=220 velocity=6.283

Commit message: add walkman WaistLat, fix plotting titles

File: model/walkman.urdf (robot description, URDF)
Before this commit: robot bigman, 86 links, 85 joints
Joints:
- joint WaistLat: limit lower=-0.610865238196 upper=0.610865238196 effort=120 velocity=6.283 -> lower=-0.3490658503988659 upper=0.3490658503988659 effort=120 velocity=6.283; type fixed -> revolute

File: model/walkman_measured.urdf (robot description, URDF)
Before this commit: robot bigman, 86 links, 85 joints
Joints:
- joint WaistLat: limit lower=-0.610865238196 upper=0.610865238196 effort=120 velocity=6.283 -> lower=-0.3490658503988659 upper=0.3490658503988659 effort=120 velocity=6.283; type fixed -> revolute

Commit message: add suspended base dynamics, fix SDP identification, improve simulator fidelity
Add ball-joint suspended dynamics simulation for floating-base identification.
The robot hangs from a configurable attachment frame (crane_ft) and base motion
is computed from Newton-Euler equations, giving the 6 base wrench equations
real information content. Integrated into both trajectory optimizer and simulator.

Fix several SDP identification issues: missing contactForcesSum in rho2_norm_sqr,
hardcoded onlyUseDSDP, checkFeasibility crash on SymPy Zero scalars, and add
configurable solver tolerances (sdpSafeMargin, sdpFeasTol).

Fix simulator: remove fabricated base motion, preserve measured base wrench,
default output to .measurements.npz to prevent overwriting trajectory files.

New config: floatingBaseAttachment (fixed/suspended/free), dontChangeLinks,
sdpSafeMargin, sdpFeasTol. Ctrl-C now cleanly terminates optimizer workers.

File: model/walkman.urdf (robot description, URDF)
Before this commit: robot bigman, 86 links, 85 joints
Links:
- link crane_ft: mass None -> 0.001

File: model/walkman_measured.urdf (robot description, URDF)
Before this commit: robot bigman, 86 links, 85 joints
Links:
- link crane_ft: mass None -> 0.001
