Commit message: two-step friction identification and friction model improvements
  Implement Ayusawa (2014) base-link approach for friction-free inertial
  parameter identification on floating-base robots. The base wrench equations
  (6 per sample) contain no joint friction terms, enabling clean inertial
  identification. A post-identification step then fits Fc, Fv, and torque
  offset per joint from the residual.

  Friction model improvements:
  - Add torque offset term (tau_off) per joint, absorbing amplifier bias and
    sensor offsets (standard in Gautier et al.)
  - Add Tikhonov regularization on friction params toward a priori values,
    preventing Fc/Fv explosion from their correlation in periodic trajectories
  - Add Stribeck friction term (disabled by default, Fc/Fs correlation)

  Other changes:
  - Rename walkman.urdf to walkman_apriori.urdf with realistic friction mismatch
    (5% of effort limit vs real 3%) for more meaningful benchmarking
  - Lower suspended dynamics damping (500 → 15 Nm·s/rad) for meaningful base
    dynamics excitation

  On the walkman benchmark (29 DOF, wrong a priori friction):
  - Base param distance: 15.3 vs 30.2 a priori (49% improvement)
  - NRMS with post-identified friction: 1.41% vs 2.67% inertial-only

File: model/world_walkman_suspended.urdf (robot description, URDF)
Before this commit: robot crane_world, 5 links, 4 joints
Links:
- link crane_arm: mass 20.0 -> 30.0; geometry visual box size=2.0 0.10 0.10
- link crane_column: geometry visual box size=0.15 0.15 2.5
Joints:
- joint crane_arm_joint: origin xyz=-0.7 0 0.25 rpy=0 0 0 -> xyz=-1.2 0 0.25 rpy=0 0 0
- joint crane_column_joint: origin xyz=-0.7 0 -2.2 rpy=0 0 0 -> xyz=-1.2 0 -2.2 rpy=0 0 0
