Commit message: more realistic walkman torque noise, more pertubation of a priori parameters for testing identification

File: model/walkman_apriori.urdf (robot description, URDF)
Before this commit: robot bigman, 86 links, 85 joints
Links:
- link DWL: mass 1.44965471 -> 1.62393960
- link DWS: mass 5.28825567 -> 5.82188154
- link DWYTorso: mass 26 -> 8.03384087
- link LElb: mass 8.6765385e-01 -> 0.77275176
- link LFoot: mass 3.42638110 -> 2.28980943
- link LFootmot: mass 3.2844159 -> 3.07375923
- link LForearm: mass 2.2127686 -> 2.09446476
- link LHipMot: mass 3.7958197 -> 3.50029395
- link LLowLeg: mass 5.6495309 -> 6.32817416
- link LShp: mass 1.81745527 -> 1.59833920
- link LShr: mass 5.00486460 -> 4.71203907
- link LShy: mass 3.20289133 -> 3.19885974
- link LSoftHandLink: mass 1.2 -> 2.36330972
- link LThighLowLeg: mass 5.0950736 -> 5.35135688
- link LThighUpLeg: mass 3.2402068 -> 2.66176684
- link LWrMot2: mass 1.2838072 -> 1.19465445
- link LWrMot3: mass 4.2801447e-01 -> 0.16270568
- link NeckPitch: mass 0.623 -> 0.15425476
- link NeckYaw: mass 0.35 -> 0.45891713
- link RElb: mass 8.6765385e-01 -> 0.84224368
- link RFoot: mass 3.42638110 -> 2.48363431
- link RFootmot: mass 3.2844159 -> 2.75686395
- link RForearm: mass 2.2127686 -> 2.10337727
- link RHipMot: mass 3.7958197 -> 3.55380981
- link RLowLeg: mass 5.6495309 -> 5.69349708
- link RShp: mass 1.81745527 -> 1.95410466
- link RShr: mass 5.00486460 -> 5.07396915
- link RShy: mass 3.20289133 -> 3.23766656
- link RSoftHandLink: mass 1.2 -> 2.23037198
- link RThighLowLeg: mass 5.0950736 -> 5.18383457
- link RThighUpLeg: mass 3.2402068 -> 2.72753304
- link RWrMot2: mass 1.2838072 -> 1.04328337
- link RWrMot3: mass 4.2801447e-01 -> 0.16109230
- link TorsoProtections: mass 4.7 -> 4.41086969
- link Waist: mass 1.1046081e+01 -> 10.02296987
- link backpack: mass 10.0 -> 14.72519204
- link multisense/head: mass 1.41984 -> 4.06488321
- link multisense/hokuyo_link: mass 0.057654 -> 0.31059106
Joints:
- joint left_camera_frame_joint: origin xyz=0.0 0.035 -0.002 -> xyz=-0.02787746 0.00379130 -0.02191020
